Commit message: Turn on boundaries

File: object/boundary_long.urdf (robot description, URDF)
Before this commit: robot wall, 1 links, 0 joints
Links:
- link baseLink: geometry collision box size=16 10 1; visual mesh filename=boundary_long.obj scale=1 1 1

File: object/boundary_short.urdf (robot description, URDF)
Before this commit: robot wall, 1 links, 0 joints
Links:
- link baseLink: geometry collision box size=1 10 9; visual mesh filename=boundary_short.obj scale=1 1 1
